File: apple-ii-8t28-74ls245-adapter/apple-ii-8t28-74ls245-adapter.sch (KiCad schematic (older format))
At the start: 4 parts, among them J1 8T28 H11, J2 8T28 H10, U1 74LS245

Commit message: More layout fixes
Parts:
- C1: footprint (none) -> Capacitor_THT:C_Axial_L3.8mm_D2.6mm_P7.50mm_Horizontal
- J1, J2: footprint (none) -> Package_DIP:DIP-16_W7.62mm_Socket
- U1: footprint (none) -> Package_DIP:DIP-20_W7.62mm_Socket
Changed lines of the file:
@@
 F 0 "U1" H 3900 3031 50  0000 C CNN
 F 1 "74LS245" H 3900 2940 50  0000 C CNN
-F 2 "" H 3900 2050 50  0001 C CNN
+F 2 "Package_DIP:DIP-20_W7.62mm_Socket" H 3900 2050 50  0001 C CNN
 F 3 "http://www.ti.com/lit/gpn/sn74LS245" H 3900 2050 50  0001 C CNN
 	1    3900 2050
@@
 F 0 "C1" H 5192 3446 50  0000 L CNN
 F 1 "0.1uF" H 5192 3355 50  0000 L CNN
-F 2 "" H 5100 3400 50  0001 C CNN
+F 2 "Capacitor_THT:C_Axial_L3.8mm_D2.6mm_P7.50mm_Horizontal" H 5100 3400 50  0001 C CNN
 F 3 "~" H 5100 3400 50  0001 C CNN
 	1    5100 3400
@@
 F 0 "J1" H 2750 5117 50  0000 C CNN
 F 1 "8T28 H11" H 2750 5026 50  0000 C CNN
-F 2 "" H 2700 4600 50  0001 C CNN
+F 2 "Package_DIP:DIP-16_W7.62mm_Socket" H 2700 4600 50  0001 C CNN
 F 3 "~" H 2700 4600 50  0001 C CNN
 	1    2700 4600
@@
 F 0 "J2" H 4350 5117 50  0000 C CNN
 F 1 "8T28 H10" H 4350 5026 50  0000 C CNN
-F 2 "" H 4300 4600 50  0001 C CNN
+F 2 "Package_DIP:DIP-16_W7.62mm_Socket" H 4300 4600 50  0001 C CNN
 F 3 "~" H 4300 4600 50  0001 C CNN
 	1    4300 4600
@@
 $EndComp
 $Comp
-L power:GND #PWR?
+L power:GND #PWR0101
 U 1 1 60C8437D
 P 2500 5000
-F 0 "#PWR?" H 2500 4750 50  0001 C CNN
+F 0 "#PWR0101" H 2500 4750 50  0001 C CNN
 F 1 "GND" H 2505 4827 50  0000 C CNN
 F 2 "" H 2500 5000 50  0001 C CNN
@@
 $EndComp
 $Comp
-L power:GND #PWR?
+L power:GND #PWR0102
 U 1 1 60C846EA
 P 4100 5000
-F 0 "#PWR?" H 4100 4750 50  0001 C CNN
+F 0 "#PWR0102" H 4100 4750 50  0001 C CNN
 F 1 "GND" H 4105 4827 50  0000 C CNN
 F 2 "" H 4100 5000 50  0001 C CNN
@@
 $EndComp
 $Comp
-L power:VCC #PWR?
+L power:VCC #PWR0103
 U 1 1 60C84A5F
 P 3000 4300
-F 0 "#PWR?" H 3000 4150 50  0001 C CNN
+F 0 "#PWR0103" H 3000 4150 50  0001 C CNN
 F 1 "VCC" H 3015 4473 50  0000 C CNN
 F 2 "" H 3000 4300 50  0001 C CNN
@@
 $EndComp
 $Comp
-L power:VCC #PWR?
+L power:VCC #PWR0104
 U 1 1 60C84EC4
 P 4600 4300
-F 0 "#PWR?" H 4600 4150 50  0001 C CNN
+F 0 "#PWR0104" H 4600 4150 50  0001 C CNN
 F 1 "VCC" H 4615 4473 50  0000 C CNN
 F 2 "" H 4600 4300 50  0001 C CNN
@@
 $EndComp
 $Comp
-L power:GND #PWR?
+L power:GND #PWR0105
 U 1 1 60C85653
 P 3900 2850
-F 0 "#PWR?" H 3900 2600 50  0001 C CNN
+F 0 "#PWR0105" H 3900 2600 50  0001 C CNN
 F 1 "GND" H 3905 2677 50  0000 C CNN
 F 2 "" H 3900 2850 50  0001 C CNN
@@
 $EndComp
 $Comp
-L power:VCC #PWR?
+L power:VCC #PWR0106
 U 1 1 60C85B98
 P 3900 1250
-F 0 "#PWR?" H 3900 1100 50  0001 C CNN
+F 0 "#PWR0106" H 3900 1100 50  0001 C CNN
 F 1 "VCC" H 3915 1423 50  0000 C CNN
 F 2 "" H 3900 1250 50  0001 C CNN
@@
 $EndComp
 $Comp
-L power:GND #PWR?
+L power:GND #PWR0107
 U 1 1 60C8CFCB
 P 5100 3500
-F 0 "#PWR?" H 5100 3250 50  0001 C CNN
+F 0 "#PWR0107" H 5100 3250 50  0001 C CNN
 F 1 "GND" H 5105 3327 50  0000 C CNN
 F 2 "" H 5100 3500 50  0001 C CNN
@@
 $EndComp
 $Comp
-L power:VCC #PWR?
+L power:VCC #PWR0108
 U 1 1 60C8D2F8
 P 5100 3300
-F 0 "#PWR?" H 5100 3150 50  0001 C CNN
+F 0 "#PWR0108" H 5100 3150 50  0001 C CNN
 F 1 "VCC" H 5115 3473 50  0000 C CNN
 F 2 "" H 5100 3300 50  0001 C CNN
@@
 CPU_DIR
 $Comp
-L power:GND #PWR?
+L power:GND #PWR0109
 U 1 1 60C9B21D
 P 3400 2550
-F 0 "#PWR?" H 3400 2300 50  0001 C CNN
+F 0 "#PWR0109" H 3400 2300 50  0001 C CNN
 F 1 "GND" H 3405 2377 50  0000 C CNN
 F 2 "" H 3400 2550 50  0001 C CNN
