File: ubitx-mixer-filter-board/ubitx-mixer-filter-board.sch (KiCad schematic (older format))
At the start: 45 parts, among them J1 CLOCK, J2 UNBALANCE, J3 OUTPUT_A, J4 OUTPUT_B, Y1 45.15MHz

Commit message: Update schematic and board layout a bit, I still need to finish this!
Parts:
- renumbered D1 to D3
Other:
- note added: "30MHz LPF\n"
- note added: "45.15MHz IF filter"
- note added: "Mixer"
- note added: "Mixer balance/unbalance control"
Changed lines of the file:
@@
 Connection ~ 2750 2750
 $Comp
-L power:GND #PWR?
+L power:GND #PWR0101
 U 1 1 60505034
 P 2750 2750
-F 0 "#PWR?" H 2750 2500 50  0001 C CNN
+F 0 "#PWR0101" H 2750 2500 50  0001 C CNN
 F 1 "GND" H 2755 2577 50  0000 C CNN
 F 2 "" H 2750 2750 50  0001 C CNN
@@
 	2550 2100 2550 2150
 $Comp
-L power:GND #PWR?
+L power:GND #PWR0102
 U 1 1 6052152F
 P 2300 2100
-F 0 "#PWR?" H 2300 1850 50  0001 C CNN
+F 0 "#PWR0102" H 2300 1850 50  0001 C CNN
 F 1 "GND" H 2305 1927 50  0000 C CNN
 F 2 "" H 2300 2100 50  0001 C CNN
@@
 Connection ~ 3000 5100
 $Comp
-L power:GND #PWR?
+L power:GND #PWR0103
 U 1 1 6061C372
 P 2600 5300
-F 0 "#PWR?" H 2600 5050 50  0001 C CNN
+F 0 "#PWR0103" H 2600 5050 50  0001 C CNN
 F 1 "GND" H 2605 5127 50  0000 C CNN
 F 2 "" H 2600 5300 50  0001 C CNN
@@
 $EndComp
 $Comp
-L power:GND #PWR?
+L power:GND #PWR0104
 U 1 1 6061C9C8
 P 3000 5300
-F 0 "#PWR?" H 3000 5050 50  0001 C CNN
+F 0 "#PWR0104" H 3000 5050 50  0001 C CNN
 F 1 "GND" H 3005 5127 50  0000 C CNN
 F 2 "" H 3000 5300 50  0001 C CNN
@@
 $EndComp
 $Comp
-L power:GND #PWR?
+L power:GND #PWR0105
 U 1 1 606E7A0D
 P 5500 2100
-F 0 "#PWR?" H 5500 1850 50  0001 C CNN
+F 0 "#PWR0105" H 5500 1850 50  0001 C CNN
 F 1 "GND" H 5505 1927 50  0000 C CNN
 F 2 "" H 5500 2100 50  0001 C CNN
@@
 $EndComp
 $Comp
-L power:GND #PWR?
+L power:GND #PWR0106
 U 1 1 606E81B3
 P 6500 2100
-F 0 "#PWR?" H 6500 1850 50  0001 C CNN
+F 0 "#PWR0106" H 6500 1850 50  0001 C CNN
 F 1 "GND" H 6505 1927 50  0000 C CNN
 F 2 "" H 6500 2100 50  0001 C CNN
@@
 $EndComp
 $Comp
-L power:GND #PWR?
+L power:GND #PWR0107
 U 1 1 606E8BBC
 P 6000 2100
-F 0 "#PWR?" H 6000 1850 50  0001 C CNN
+F 0 "#PWR0107" H 6000 1850 50  0001 C CNN
 F 1 "GND" H 6005 1927 50  0000 C CNN
 F 2 "" H 6000 2100 50  0001 C CNN
@@
 $EndComp
 $Comp
-L power:GND #PWR?
+L power:GND #PWR0108
 U 1 1 606E939A
 P 7000 2100
-F 0 "#PWR?" H 7000 1850 50  0001 C CNN
+F 0 "#PWR0108" H 7000 1850 50  0001 C CNN
 F 1 "GND" H 7005 1927 50  0000 C CNN
 F 2 "" H 7000 2100 50  0001 C CNN
@@
 $EndComp
 $Comp
-L power:GND #PWR?
+L power:GND #PWR0109
 U 1 1 606E9B8F
 P 7500 2100
-F 0 "#PWR?" H 7500 1850 50  0001 C CNN
+F 0 "#PWR0109" H 7500 1850 50  0001 C CNN
 F 1 "GND" H 7505 1927 50  0000 C CNN
 F 2 "" H 7500 2100 50  0001 C CNN
@@
 	5750 4400 5850 4400
 $Comp
-L power:GND #PWR?
+L power:GND #PWR0110
 U 1 1 60717B9A
 P 5750 4600
-F 0 "#PWR?" H 5750 4350 50  0001 C CNN
+F 0 "#PWR0110" H 5750 4350 50  0001 C CNN
 F 1 "GND" H 5755 4427 50  0000 C CNN
 F 2 "" H 5750 4600 50  0001 C CNN
@@
 $EndComp
 $Comp
-L power:GND #PWR?
+L power:GND #PWR0111
 U 1 1 607497E2
 P 5400 3250
-F 0 "#PWR?" H 5400 3000 50  0001 C CNN
+F 0 "#PWR0111" H 5400 3000 50  0001 C CNN
 F 1 "GND" H 5405 3077 50  0000 C CNN
 F 2 "" H 5400 3250 50  0001 C CNN
@@
 $EndComp
 $Comp
-L power:GND #PWR?
+L power:GND #PWR0112
 U 1 1 60749E04
 P 6200 3250
-F 0 "#PWR?" H 6200 3000 50  0001 C CNN
+F 0 "#PWR0112" H 6200 3000 50  0001 C CNN
 F 1 "GND" H 6205 3077 50  0000 C CNN
 F 2 "" H 6200 3250 50  0001 C CNN
@@
 $EndComp
 $Comp
-L power:GND #PWR?
+L power:GND #PWR0113
 U 1 1 6074A435
 P 6550 3350
-F 0 "#PWR?" H 6550 3100 50  0001 C CNN
+F 0 "#PWR0113" H 6550 3100 50  0001 C CNN
 F 1 "GND" H 6555 3177 50  0000 C CNN
 F 2 "" H 6550 3350 50  0001 C CNN
@@
 $EndComp
 $Comp
-L power:GND #PWR?
+L power:GND #PWR0114
 U 1 1 6074AA7A
 P 6900 3250
-F 0 "#PWR?" H 6900 3000 50  0001 C CNN
+F 0 "#PWR0114" H 6900 3000 50  0001 C CNN
 F 1 "GND" H 6905 3077 50  0000 C CNN
 F 2 "" H 6900 3250 50  0001 C CNN
@@
 $EndComp
 $Comp
-L power:GND #PWR?
+L power:GND #PWR0115
 U 1 1 6074B0D3
 P 7700 3250
-F 0 "#PWR?" H 7700 3000 50  0001 C CNN
+F 0 "#PWR0115" H 7700 3000 50  0001 C CNN
 F 1 "GND" H 7705 3077 50  0000 C CNN
 F 2 "" H 7700 3250 50  0001 C CNN
@@
 OUTPUT_B
 $Comp
-L Device:D D1
+L Device:D D3
 U 1 1 60772C5E
 P 6300 4400
-F 0 "D1" H 6300 4183 50  0000 C CNN
+F 0 "D3" H 6300 4183 50  0000 C CNN
 F 1 "1N4148" H 6300 4274 50  0000 C CNN
 F 2 "" H 6300 4400 50  0001 C CNN
@@
 $EndComp
 $Comp
-L power:GND #PWR?
+L power:GND #PWR0116
 U 1 1 607BC32E
 P 5050 5500
-F 0 "#PWR?" H 5050 5250 50  0001 C CNN
+F 0 "#PWR0116" H 5050 5250 50  0001 C CNN
 F 1 "GND" H 5055 5327 50  0000 C CNN
 F 2 "" H 5050 5500 50  0001 C CNN
@@
 $EndComp
 $Comp
-L power:GND #PWR?
+L power:GND #PWR0117
 U 1 1 607C3371
 P 5050 6100
-F 0 "#PWR?" H 5050 5850 50  0001 C CNN
+F 0 "#PWR0117" H 5050 5850 50  0001 C CNN
 F 1 "GND" H 5055 5927 50  0000 C CNN
 F 2 "" H 5050 6100 50  0001 C CNN
@@
 $EndComp
 $Comp
-L power:GND #PWR?
+L power:GND #PWR0118
 U 1 1 60806C47
 P 6650 6100
-F 0 "#PWR?" H 6650 5850 50  0001 C CNN
+F 0 "#PWR0118" H 6650 5850 50  0001 C CNN
 F 1 "GND" H 6655 5927 50  0000 C CNN
 F 2 "" H 6650 6100 50  0001 C CNN
@@
 $EndComp
 $Comp
-L power:GND #PWR?
+L power:GND #PWR0119
 U 1 1 608071C1
 P 6650 5500
-F 0 "#PWR?" H 6650 5250 50  0001 C CNN
+F 0 "#PWR0119" H 6650 5250 50  0001 C CNN
 F 1 "GND" H 6655 5327 50  0000 C CNN
 F 2 "" H 6650 5500 50  0001 C CNN
@@
 Text GLabel 6650 5400 2    50   Input ~ 0
 OUTPUT_B
+Text Notes 1800 2500 0    50   ~ 0
+Mixer
+Text Notes 5200 1500 0    50   ~ 0
+30MHz LPF\n
+Text Notes 5200 2700 0    50   ~ 0
+45.15MHz IF filter
+Text Notes 5150 4050 0    50   ~ 0
+Mixer balance/unbalance control
 $EndSCHEMATC
