File: pcw/pcw-expansion/pcw-expansion.kicad_sch (KiCad schematic)
At the start: 16 parts, among them IC1 DART-DIP-40, J1 edge connector, J2 TTL serial, J3 parallel, J5 video out, J6 joystick, J7 composite out, J8 stereo, U1 8254, U2 AS6C4008-55PCN, U3 AS6C4008-55PCN, U4 AS6C4008-55PCN, U5 74LS374, U6 74HC00, U7 GAL16V8, U8 28C256

Commit message: [pcw] more schematic updates!
slowly but surely getting there!
Parts:
- removed U7: GAL16V8, symbol Logic_Programmable:GAL16V8
- added C1: 0.1u, symbol Device:C_Small
- added J4: video in, symbol Connector:Conn_01x04_Pin
- added J9: video mode, symbol Connector:Conn_01x03_Pin
- added R1, R4: 5.6k, symbol Device:R_Small
- added R10, R3, R5, R6, R7, R8: 1k, symbol Device:R_Small
- added R2: 470, symbol Device:R_Small
- added R9: 10k, symbol Device:R_Small
- added SW1: RESET, symbol Switch:SW_Push
- added U10, U11: GAL22V10, symbol 8bits:GAL22V10
- added U7: LM358, symbol Amplifier_Operational:LM358
- added U9: PSG_AY-3-8910, symbol 8bits:PSG_AY-3-8910
- J7: value composite out -> comp out
Connections:
- net D0: now also J1.31 (Pin_31), U9.37 (D0)
- net SYNC_OUT: now reaches J5.1 (Pin_1)
- net SYNC_OUT: now also U6.6, R3.1
- net GND: now reaches J5.2 (Pin_2)
- net GND: now also IC1.31 (GND), IC1.6 (IEI), J1.3 (Pin_3), J1.4 (Pin_4), J1.49 (Pin_49), J1.50 (Pin_50), J3.18 (P18), J3.19 (P19), J3.20 (P20), J3.21 (P21), J3.22 (P22), J3.23 (P23), J3.24 (P24), J3.25 (P25), J5.4 (Pin_4), J6.0 (PAD), J7.2 (Ext), U1.12 (GND), U2.16 (VSS), U3.16 (VSS), U4.16 (VSS), U5.1 (OE), U5.10 (GND), U6.7 (GND), U8.14 (GND), C1.2, J4.2 (Pin_2), J4.4 (Pin_4), J9.3 (Pin_3), R1.1, SW1.1, U10.12 (GND), U11.12 (GND), U7.4 (V-), U9.1 (Vss)
- net VIDEO_OUT: now reaches J5.3 (Pin_3)
- net VIDEO_OUT: now also U6.3, R2.1
- net at U6.4: now also U6.8
- net +5V: now reaches U6.5
- net +5V: now also IC1.9 (+5V), J1.5 (Pin_5), J1.6 (Pin_6), U1.24 (VCC), U2.32 (VCC), U3.32 (VCC), U4.32 (VCC), U5.20 (VCC), U6.12, U6.14 (VCC), U6.2, U6.9, U8.28 (VCC), C1.1, J9.1 (Pin_1), R10.1, R6.2, R7.2, R8.2, U10.24 (VCC), U11.24 (VCC), U9.40 (Vcc)
- net D1: now reaches U3.14 (DQ1)
- net D1: now also IC1.1 (D1), J1.32 (Pin_32), U1.7 (D1), U2.14 (DQ1), U4.14 (DQ1), U5.4 (D1), U8.12 (D1), U9.36 (D1)
- net D2: now reaches U3.15 (DQ2)
- net D2: now also IC1.39 (D2), J1.29 (Pin_29), U1.6 (D2), U2.15 (DQ2), U4.15 (DQ2), U5.7 (D2), U8.13 (D2), U9.35 (D2)
- net D3: now reaches U3.17 (DQ3)
- net D3: now also IC1.2 (D3), J1.30 (Pin_30), U1.5 (D3), U2.17 (DQ3), U4.17 (DQ3), U5.8 (D3), U8.15 (D3), U9.34 (D3)
- net D4: now reaches U3.18 (DQ4)
- net D4: now also IC1.38 (D4), J1.27 (Pin_27), U1.4 (D4), U2.18 (DQ4), U4.18 (DQ4), U5.13 (D4), U8.16 (D4), U9.33 (D4)
- net D5: now reaches U3.19 (DQ5)
- net D5: now also IC1.3 (D5), J1.28 (Pin_28), U1.3 (D5), U2.19 (DQ5), U4.19 (DQ5), U5.14 (D5), U8.17 (D5), U9.32 (D5)
- net D6: now reaches U3.20 (DQ6)
- net D6: now also IC1.37 (D6), J1.25 (Pin_25), U1.2 (D6), U2.20 (DQ6), U4.20 (DQ6), U5.17 (D6), U8.18 (D6), U9.31 (D6)
- net D7: now reaches U3.21 (DQ7)
- net D7: now also IC1.4 (D7), J1.26 (Pin_26), U1.1 (D7), U2.21 (DQ7), U4.21 (DQ7), U5.18 (D7), U8.19 (D7), U9.30 (D7)
- net SYNC_IN: now reaches U6.10
- net SYNC_IN: now also J4.1 (Pin_1), R4.2
- net /CEN_STROBE: now reaches J3.1
- net CEN_BUSY: now reaches J3.11
- net CEN_BUSY: now also R10.2, R9.1
- net CEN_D0: now reaches J3.2
- net CEN_D0: now also U5.2 (O0)
- net CEN_D1: now reaches J3.3
- net CEN_D1: now also U5.5 (O1)
- net CEN_D2: now reaches J3.4
- net CEN_D2: now also U5.6 (O2)
- net CEN_D3: now reaches J3.5
- net CEN_D3: now also U5.9 (O3)
- net CEN_D4: now reaches J3.6
- net CEN_D4: now also U5.12 (O4)
- net CEN_D5: now reaches J3.7
- net CEN_D5: now also U5.15 (O5)
- net CEN_D6: now reaches J3.8
- net CEN_D6: now also U5.16 (O6)
- net CEN_D7: now reaches J3.9
- net CEN_D7: now also U5.19 (O7)
- net at U6.11: now also U6.1
- net VIDEO_IN: now reaches U6.13
- net VIDEO_IN: now also J4.3 (Pin_3), R1.2
- net /PRT_CS: now reaches U5.11 (Cp)
- net UART_CLK_2: now reaches IC1.13 (~{RXCA})
- net UART_CLK_2: now also U1.13 (OUT1)
- net UART_CLK_1: now reaches IC1.14 (~{TXCA})
- net UART_CLK_1: now also U1.10 (OUT0)
- net 4MHZ: now reaches IC1.20 (Φ)
- net 4MHZ: now also J1.48 (Pin_48)
- net /RESET: now reaches IC1.21 (~{RESET})
- net /RESET: now also J1.33 (Pin_33), R5.2, U9.23 (~{RESET})
- net /UART_CTSB: now reaches IC1.23 (~{CTSB})
- net /UART_CTSB: now also R9.2
- net /UART_DTRB: now reaches IC1.25 (~{DTRB})
- net UART_CLK_3: now reaches IC1.27 (~{RxTxCB})
- net UART_CLK_3: now also U1.17 (OUT2)
- net /RD: now reaches IC1.32 (~{RD})
- net /RD: now also J1.41 (Pin_41), U1.22 (~{RD})
- net A0: now reaches IC1.33 (C/~{D})
- net A0: now also J1.23 (Pin_23), U1.19 (A0)
- net A1: now reaches IC1.34 (B/~{A})
- net A1: now also J1.24 (Pin_24), U1.20 (A1)
- net /DART_CS: now reaches IC1.35 (~{CE})
- net /IORQ: now reaches IC1.36 (~{IORQ})
- net /IORQ: now also J1.42 (Pin_42)
- net /INT: now reaches IC1.5 (~{INT})
- net /INT: now also J1.36 (Pin_36)
- net /M1: now reaches IC1.8 (~{M1})
- net /M1: now also J1.34 (Pin_34)
- net at U1.11 (G0): now also R7.1
- net at U1.14 (G1): now also R6.1
- net 2MHZ: now reaches U1.15 (CLK1)
- net 2MHZ: now also U1.18 (CLK2), U1.9 (CLK0)
- net at U1.16 (G2): now also R8.1
- net /8254_CS: now reaches U1.21 (~{CS})
- net /WR: now reaches U1.23 (~{WR})
- net /WR: now also J1.39 (Pin_39)
- net A15: now reaches J1.10 (Pin_10)
- net A12: now reaches J1.11 (Pin_11)
- net A13: now reaches J1.12 (Pin_12)
- net A10: now reaches J1.13 (Pin_13)
- net A11: now reaches J1.14 (Pin_14)
- net A8: now reaches J1.15 (Pin_15)
- net A9: now reaches J1.16 (Pin_16)
- net A6: now reaches J1.17 (Pin_17)
- net A7: now reaches J1.18 (Pin_18)
- net A4: now reaches J1.19 (Pin_19)
- net A5: now reaches J1.20 (Pin_20)
- net A2: now reaches J1.21 (Pin_21)
- net A3: now reaches J1.22 (Pin_22)
- net /BUSRQ: now reaches J1.35 (Pin_35)
- net /BUSAK: now reaches J1.37 (Pin_37)
- net /WAIT: now reaches J1.38 (Pin_38)
- net /MREQ: now reaches J1.40 (Pin_40)
- net SYNC: now reaches J1.44 (Pin_44)
- net /MDIS: now reaches J1.45 (Pin_45)
- net VIDEO: now reaches J1.46 (Pin_46)
- net 32MHZ: now reaches J1.47 (Pin_47)
- net +12V: now reaches J1.8 (Pin_8)
- net A14: now reaches J1.9 (Pin_9)
- net COMP_OUT: now reaches J7.1 (In)
- net COMP_OUT: now also R2.2, R3.2
- new net: R5.1, SW1.2
- new net VID_MODE: J9.2 (Pin_2), R4.1
Other:
- note added: "RAM: IO WR 111100xx (0xF0 -> 0xF3) These control each 16k region (0x0000, 0x4000, 0x8000, 0xC0000) RAM bank value: 0xxxxxxx - ("standard") standard RAM banking, Amstrad CPC style if this is set, don't select any RAM! RAM bank value: 1xxxxxxx (0..127) these map to physical address bits A14..A21) RAM map control: IO WR 11111011 (0xF4) a "1" in bits 4..7 controls whether "standard" RAM (bank values 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"
- note added: "UART: IO RD/WR 111000xx (0xE0 -> 0xE3) 8254: IO RD/WR 111001xx (0xE4 -> 0xE7) LS374 (Printer): IO WR 11101000 (0xE8)"
- moved on the sheet: IC1, J1, J5, J7, J8, U1, U2, U3, U4, U5, U6A, U6B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
